Commit message: Adding r2 robot.

File: catkin_ws/src/pan_tilt_description/urdf/box.urdf (robot description, URDF)
Before this commit: robot myfirst, 1 links, 0 joints
Links:
- added link world
- link base_link: mass None -> 1; geometry collision box size=0.6 0.1 0.2; visual box size=3 0.1 0.2
Joints:
- added joint fixed: type fixed, parent world, child base_link
