Commit message: Adding a second camera with driver. However, still cannot capture image stream.

File: catkin_ws/src/pan_tilt_description/urdf/pan_tilt.urdf (robot description, URDF)
Before this commit: robot pan_tilt, 4 links, 3 joints
Links:
- removed link camera_link
- added link camera_link_left, mass 1e-5; collision box size=0.025 0.025 0.025; visual box size=0.025 0.025 0.025
- added link camera_link_right, mass 1e-5; collision box size=0.025 0.025 0.025; visual box size=0.025 0.025 0.025
Joints:
- removed joint cam_to_head
- added joint left_cam_to_head: type fixed, parent head_link, child camera_link_left, origin xyz=0.063 -0.035 0.035 rpy=0 0 0, axis 0 1 0
- added joint right_cam_to_head: type fixed, parent head_link, child camera_link_right, origin xyz=0.063 -0.035 0.035 rpy=0 0 0, axis 0 1 0

File: catkin_ws/src/pan_tilt_description/urdf/pan_tilt.urdf.xacro (robot description, xacro)
@@ -89,6 +89,6 @@
     </inertial>
   </link>
-  <!-- Description of camera. -->
-  <link name="camera_link">
+  <!-- Description of right camera. -->
+  <link name="camera_link_right">
     <collision>
       <geometry>
@@ -108,11 +108,39 @@
     </inertial>
   </link>
-  <!-- Attach camera to head. -->
-  <joint name="cam_to_head" type="fixed">
+  <!-- Description of left camera. -->
+  <link name="camera_link_left">
+    <collision>
+      <geometry>
+        <box size="${camera_link} ${camera_link} ${camera_link}"/>
+      </geometry>
+    </collision>
+    <visual>
+      <geometry>
+         <box size="${camera_link} ${camera_link} ${camera_link}"/>
+      </geometry>
+      <origin rpy="0 1.57075 0" xyz="0.025 0.070 0"/>
+       <material name="blue" />
+    </visual>
+    <inertial>
+      <mass value="1e-5" />
+      <inertia ixx="1e-6" ixy="0" ixz="0" iyy="1e-6" iyz="0" izz="1e-6" />
+      <origin xyz="0 0 0" rpy="0 0 0" />
+    </inertial>
+  </link>
+  <!-- Attach right camera to head. -->
+  <joint name="right_cam_to_head" type="fixed">
     <axis xyz="0 1 0" />
     <!-- Determine measurements xyz. -->
     <origin rpy="0 0 0" xyz="0.063 -0.035 0.035" />
     <parent link="head_link" />
-    <child link="camera_link" />
+    <child link="camera_link_right" />
+  </joint>
+  <!-- Attach left camera to head. -->
+  <joint name="left_cam_to_head" type="fixed">
+    <axis xyz="0 1 0" />
+    <!-- Determine measurements xyz. -->
+    <origin rpy="0 0 0" xyz="0.063 -0.035 0.035" />
+    <parent link="head_link" />
+    <child link="camera_link_left" />
   </joint>
   <!-- Attach base to world. -->

Commit message: Adding joint to head capable of rotation

File: catkin_ws/src/pan_tilt_description/urdf/pan_tilt.urdf (robot description, URDF)
Before this commit: robot pan_tilt, 5 links, 4 joints
Joints:
- joint head_to_base: axis (none) -> 0 0 1; limit (none) -> lower=0.0 upper=3.1412 effort=1000.0 velocity=0.5; type fixed -> revolute

Commit message: Adding motion planning, robot neck can now turn

File: catkin_ws/src/pan_tilt_description/urdf/pan_tilt.urdf (robot description, URDF)
Before this commit: robot pan_tilt, 5 links, 4 joints
Joints:
- joint head_to_base: limit lower=0.0 upper=3.1412 effort=1000.0 velocity=0.5 -> lower=-1.571 upper=1.571 effort=1000.0 velocity=0.5
