Commit message: Removing r2 files and adding rviz launch files for pan_tilt.

File: catkin_ws/src/pan_tilt_description/urdf/pan_tilt.urdf.xacro (robot description, xacro)
@@ -1,4 +1,4 @@
 <?xml version="1.0"?>
-<robot name="box">
+<robot xmlns:xacro="http://www.ros.org/wiki/xacro" name="pan_tilt">
   <link name="world"/>
   <link name="base_link">
@@ -11,6 +11,7 @@
     <visual>
       <geometry>
-        <box size="3 0.1 0.2"/>
+        <box size="0.6 0.1 0.2"/>
       </geometry>
+      <origin rpy="0 1.57075 0" xyz="0 0 -0.3"/>
     </visual>
     <inertial>

Commit message: Moving position of box so that it now rests on top of plane.

File: catkin_ws/src/pan_tilt_description/urdf/pan_tilt.urdf.xacro (robot description, xacro)
@@ -13,5 +13,5 @@
         <box size="0.6 0.1 0.2"/>
       </geometry>
-      <origin rpy="0 1.57075 0" xyz="0 0 -0.3"/>
+      <origin rpy="0 1.57075 0" xyz="0 0 0.3"/>
     </visual>
     <inertial>

Commit message: Adding a camera link.

File: catkin_ws/src/pan_tilt_description/urdf/pan_tilt.urdf.xacro (robot description, xacro)
@@ -1,5 +1,11 @@
 <?xml version="1.0"?>
 <robot xmlns:xacro="http://www.ros.org/wiki/xacro" name="pan_tilt">
+  <!-- Documentation on URDF: http://wiki.ros.org/urdf/XML -->
+  <!-- Documentation on Xacro: http://wiki.ros.org/xacro -->
+  <!-- Xacro properties are constants. -->
+  <!-- Size of square 'camera' box -->
+  <xacro:property name="camera_link" value="0.05" />
   <link name="world"/>
+  <!-- Description of base. -->
   <link name="base_link">
     <collision>
@@ -11,5 +17,8 @@
     <visual>
       <geometry>
-        <box size="0.6 0.1 0.2"/>
+      <!-- http://wiki.ros.org/rviz/DisplayTypes/Axes -->
+      <!-- Red, Green, Blue -->
+      <!-- x, y, z -->
+        <box size="0.6 0.3 0.3"/>
       </geometry>
       <origin rpy="0 1.57075 0" xyz="0 0 0.3"/>
@@ -24,10 +33,70 @@
     </inertial>
   </link>
+  <!-- Description of head. -->
+  <link name="top_head">
+    <visual>
+      <geometry>
+        <box size="0.15 0.15 0.15" />
+      </geometry>
+      <origin rpy="0 1.57075 0" xyz="0 0 0.9"/>
+    </visual>
+    <collision>
+      <geometry>
+        <box size="0.15 0.15 0.15" />
+      </geometry>
+      <origin rpy="0 1.57075 0" xyz="0 0 0.9"/>
+    </collision>
+  </link>
+  <!-- Description of camera. -->
+  <link name="camera_link">
+    <collision>
+      <origin xyz="0 0 0" rpy="0 0 0" />
+      <geometry>
+        <box size="${camera_link} ${camera_link} ${camera_link}"/>
+      </geometry>
+    </collision>
+    <visual>
+      <origin xyz="0 0 0" rpy="0 0 0"/>
+      <geometry>
+         <box size="${camera_link} ${camera_link} ${camera_link}"/>
+      </geometry>
+    </visual>
+    <inertial>
+      <mass value="1e-5" />
+      <origin xyz="0 0 0" rpy="0 0 0" />
+      <!-- <inertia ixx="1e-6" ixy="0" ixz="0" iyy="1e-6" izy="0" izz="1e-6" /> -->
+      <inertia ixx="1e-6" ixy="0" ixz="0" iyy="1e-6" iyz="0" izz="1e-6" />
+    </inertial>
+  </link>
+  <!-- Attach camera to head. -->
+  <joint name="camera_joint" type="fixed">
+    <axis xyz="0 1 0" />
+    <!-- Determine measurements xyz. -->
+    <origin xyz="${camera_link} 0 0" rpy="0 0 0"/>
+    <parent link="top_head" />
+    <child link="camera_link" />
+  </joint>
+  <!-- Attach base to world. -->
   <joint name="fixed" type="fixed">
     <parent link="world"/>
     <child link="base_link"/>
   </joint>
+  <!-- Roll is around x, yaw is around z, and pitch is around y. -->
+  <!-- Connect head with base which allows the head to move in 3D. -->
+  <joint name="base_to_top_head" type="fixed">
+    <origin xyz="0 0 0.89" />
+    <parent link="base_link" />
+    <child link="top_head" />
+  </joint>
+  <!-- Make color of body and head red. -->
   <gazebo reference="base_link">
-    <material>Gazebo/Orange</material>
+    <material>Gazebo/DarkYellow</material>
+  </gazebo>
+  <gazebo reference="top_head">
+    <material>Gazebo/White</material>
+  </gazebo>
+  <!-- Make colour of camera red. -->
+  <gazebo reference="camera_link">
+    <material>Gazebo/Red</material>
   </gazebo>
 </robot>

Commit message: Fixing dimensions of base_link collision.

File: catkin_ws/src/pan_tilt_description/urdf/pan_tilt.urdf.xacro (robot description, xacro)
@@ -10,8 +10,8 @@
   <link name="base_link">
     <collision>
-      <origin xyz="0 0 0" rpy="0 0 0"/>
       <geometry>
-        <box size="0.6 0.1 0.2"/>
+        <box size="0.6 0.3 0.3"/>
       </geometry>
+      <origin rpy="0 1.57075 0" xyz="0 0 0.3"/>
     </collision>
     <visual>

Commit message: Placing head link immediately above base.

File: catkin_ws/src/pan_tilt_description/urdf/pan_tilt.urdf.xacro (robot description, xacro)
@@ -6,4 +6,21 @@
   <!-- Size of square 'camera' box -->
   <xacro:property name="camera_link" value="0.05" />
+  <!-- Dimensions of base. -->
+  <xacro:property name="base_link_size_x" value="0.6" />
+  <xacro:property name="base_link_size_y" value="0.3" />
+  <xacro:property name="base_link_size_z" value="0.3"/>
+  <!-- Dimensions of head. -->
+  <xacro:property name="head_link_size_x" value="0.15" />
+  <xacro:property name="head_link_size_y" value="0.15" />
+  <xacro:property name="head_link_size_z" value="0.15" />
+  <!-- Origin position of head.  -->
+  <!--
+    *BUG*:
+    For some mysterious reason, even when all values are 0,
+    the link refuses to stay grounded and floats above base.
+  -->
+  <xacro:property name="head_link_origin_x" value="0" />
+  <xacro:property name="head_link_origin_y" value="0" />
+  <xacro:property name="head_link_origin_z" value="0" />
   <link name="world"/>
   <!-- Description of base. -->
@@ -11,5 +28,5 @@
     <collision>
       <geometry>
-        <box size="0.6 0.3 0.3"/>
+        <box size="${base_link_size_x} ${base_link_size_y} ${base_link_size_z}"/>
       </geometry>
       <origin rpy="0 1.57075 0" xyz="0 0 0.3"/>
@@ -20,5 +37,5 @@
       <!-- Red, Green, Blue -->
       <!-- x, y, z -->
-        <box size="0.6 0.3 0.3"/>
+        <box size="${base_link_size_x} ${base_link_size_y} ${base_link_size_z}"/>
       </geometry>
       <origin rpy="0 1.57075 0" xyz="0 0 0.3"/>
@@ -34,17 +51,25 @@
   </link>
   <!-- Description of head. -->
-  <link name="top_head">
+  <link name="head_link">
+    <collision>
+      <geometry>
+        <box size="${head_link_size_x} ${head_link_size_y} ${head_link_size_z}" />
+      </geometry>
+      <origin rpy="0 1.57075 0" xyz="${head_link_origin_x} ${head_link_origin_y} ${head_link_origin_z}"/>
+    </collision>
     <visual>
       <geometry>
-        <box size="0.15 0.15 0.15" />
+        <box size="${head_link_size_x} ${head_link_size_y} ${head_link_size_z}" />
       </geometry>
-      <origin rpy="0 1.57075 0" xyz="0 0 0.9"/>
+      <origin rpy="0 1.57075 0" xyz="${head_link_origin_x} ${head_link_origin_y} ${head_link_origin_z}"/>
     </visual>
-    <collision>
-      <geometry>
-        <box size="0.15 0.15 0.15" />
-      </geometry>
-      <origin rpy="0 1.57075 0" xyz="0 0 0.9"/>
-    </collision>
+    <inertial>
+      <origin xyz="0 0 0" rpy="0 0 0"/>
+      <mass value="1"/>
+      <inertia
+        ixx="1.0" ixy="0.0" ixz="0.0"
+        iyy="1.0" iyz="0.0"
+        izz="1.0"/>
+    </inertial>
   </link>
   <!-- Description of camera. -->
@@ -65,5 +90,4 @@
       <mass value="1e-5" />
       <origin xyz="0 0 0" rpy="0 0 0" />
-      <!-- <inertia ixx="1e-6" ixy="0" ixz="0" iyy="1e-6" izy="0" izz="1e-6" /> -->
       <inertia ixx="1e-6" ixy="0" ixz="0" iyy="1e-6" iyz="0" izz="1e-6" />
     </inertial>
@@ -74,5 +98,5 @@
     <!-- Determine measurements xyz. -->
     <origin xyz="${camera_link} 0 0" rpy="0 0 0"/>
-    <parent link="top_head" />
+    <parent link="head_link" />
     <child link="camera_link" />
   </joint>
@@ -84,8 +108,8 @@
   <!-- Roll is around x, yaw is around z, and pitch is around y. -->
   <!-- Connect head with base which allows the head to move in 3D. -->
-  <joint name="base_to_top_head" type="fixed">
-    <origin xyz="0 0 0.89" />
+  <joint name="base_to_head_link" type="fixed">
+    <origin xyz="0 0 0.68" />
     <parent link="base_link" />
-    <child link="top_head" />
+    <child link="head_link" />
   </joint>
   <!-- Make color of body and head red. -->
@@ -93,5 +117,5 @@
     <material>Gazebo/DarkYellow</material>
   </gazebo>
-  <gazebo reference="top_head">
+  <gazebo reference="head_link">
     <material>Gazebo/White</material>
   </gazebo>

Commit message: Positioning cam_1 onto head.

File: catkin_ws/src/pan_tilt_description/urdf/pan_tilt.urdf.xacro (robot description, xacro)
@@ -5,5 +5,5 @@
   <!-- Xacro properties are constants. -->
   <!-- Size of square 'camera' box -->
-  <xacro:property name="camera_link" value="0.05" />
+  <xacro:property name="camera_link" value="0.025" />
   <!-- Dimensions of base. -->
   <xacro:property name="base_link_size_x" value="0.6" />
@@ -23,4 +23,13 @@
   <xacro:property name="head_link_origin_y" value="0" />
   <xacro:property name="head_link_origin_z" value="0" />
+  <material name="blue">
+    <color rgba="0 0 0.8 1"/>
+  </material>
+  <material name="white">
+    <color rgba="1 1 1 1"/>
+  </material>
+  <material name="orange">
+    <color rgba="179.0 107.0 0.0 1.0"/>
+  </material>
   <link name="world"/>
   <!-- Description of base. -->
@@ -40,4 +49,5 @@
       </geometry>
       <origin rpy="0 1.57075 0" xyz="0 0 0.3"/>
+      <material name="white" />
     </visual>
     <inertial>
@@ -63,4 +73,5 @@
       </geometry>
       <origin rpy="0 1.57075 0" xyz="${head_link_origin_x} ${head_link_origin_y} ${head_link_origin_z}"/>
+      <material name="orange" />
     </visual>
     <inertial>
@@ -76,5 +87,4 @@
   <link name="camera_link">
     <collision>
-      <origin xyz="0 0 0" rpy="0 0 0" />
       <geometry>
         <box size="${camera_link} ${camera_link} ${camera_link}"/>
@@ -82,17 +92,17 @@
     </collision>
     <visual>
-      <origin xyz="0 0 0" rpy="0 0 0"/>
       <geometry>
          <box size="${camera_link} ${camera_link} ${camera_link}"/>
       </geometry>
+      <origin rpy="0 1.57075 0" xyz="0.063 -0.035 0.035"/>
     </visual>
     <inertial>
       <mass value="1e-5" />
+      <inertia ixx="1e-6" ixy="0" ixz="0" iyy="1e-6" iyz="0" izz="1e-6" />
       <origin xyz="0 0 0" rpy="0 0 0" />
-      <inertia ixx="1e-6" ixy="0" ixz="0" iyy="1e-6" iyz="0" izz="1e-6" />
     </inertial>
   </link>
   <!-- Attach camera to head. -->
-  <joint name="camera_joint" type="fixed">
+  <joint name="head_to_cam" type="fixed">
     <axis xyz="0 1 0" />
     <!-- Determine measurements xyz. -->
@@ -100,4 +110,5 @@
     <parent link="head_link" />
     <child link="camera_link" />
+    <origin xyz="0 0 0"/>
   </joint>
   <!-- Attach base to world. -->

Commit message: Adding joint between camera and head.

File: catkin_ws/src/pan_tilt_description/urdf/pan_tilt.urdf.xacro (robot description, xacro)
@@ -95,5 +95,5 @@
          <box size="${camera_link} ${camera_link} ${camera_link}"/>
       </geometry>
-      <origin rpy="0 1.57075 0" xyz="0.063 -0.035 0.035"/>
+      <origin rpy="0 1.57075 0" xyz="0.025 0 0"/>
     </visual>
     <inertial>
@@ -107,5 +107,5 @@
     <axis xyz="0 1 0" />
     <!-- Determine measurements xyz. -->
-    <origin xyz="${camera_link} 0 0" rpy="0 0 0"/>
+    <origin rpy="0 0 0" xyz="0.063 -0.035 0.035" />
     <parent link="head_link" />
     <child link="camera_link" />

Commit message: Adding launch file for spawning URDF in Gazebo.

File: catkin_ws/src/pan_tilt_description/urdf/pan_tilt.urdf.xacro (robot description, xacro)
@@ -104,5 +104,5 @@
   </link>
   <!-- Attach camera to head. -->
-  <joint name="head_to_cam" type="fixed">
+  <joint name="cam_to_head" type="fixed">
     <axis xyz="0 1 0" />
     <!-- Determine measurements xyz. -->
@@ -110,8 +110,7 @@
     <parent link="head_link" />
     <child link="camera_link" />
-    <origin xyz="0 0 0"/>
   </joint>
   <!-- Attach base to world. -->
-  <joint name="fixed" type="fixed">
+  <joint name="base_to_world" type="fixed">
     <parent link="world"/>
     <child link="base_link"/>
@@ -119,19 +118,8 @@
   <!-- Roll is around x, yaw is around z, and pitch is around y. -->
   <!-- Connect head with base which allows the head to move in 3D. -->
-  <joint name="base_to_head_link" type="fixed">
-    <origin xyz="0 0 0.68" />
+  <joint name="head_to_base" type="fixed">
     <parent link="base_link" />
     <child link="head_link" />
+    <origin xyz="0 0 0.68" />
   </joint>
-  <!-- Make color of body and head red. -->
-  <gazebo reference="base_link">
-    <material>Gazebo/DarkYellow</material>
-  </gazebo>
-  <gazebo reference="head_link">
-    <material>Gazebo/White</material>
-  </gazebo>
-  <!-- Make colour of camera red. -->
-  <gazebo reference="camera_link">
-    <material>Gazebo/Red</material>
-  </gazebo>
 </robot>

Commit message: Adding .gazebo file as dependency to xacro description.

File: catkin_ws/src/pan_tilt_description/urdf/pan_tilt.urdf.xacro (robot description, xacro)
@@ -1,4 +1,14 @@
 <?xml version="1.0"?>
 <robot xmlns:xacro="http://www.ros.org/wiki/xacro" name="pan_tilt">
+  <!--
+  IMPORTANT!
+  If you modify this Xacro based URDF description, please run:
+  . update_urdf.sh
+  from directory:
+    pan_tilt_description/urdf/
+  to generate a new URDF.
+  The generated URDF will then be used by Gazebo to spawn the pan_tilt bot.
+  Failure to do this will result in your change being not reflected in simulation.
+  -->
   <!-- Documentation on URDF: http://wiki.ros.org/urdf/XML -->
   <!-- Documentation on Xacro: http://wiki.ros.org/xacro -->
@@ -23,13 +33,8 @@
   <xacro:property name="head_link_origin_y" value="0" />
   <xacro:property name="head_link_origin_z" value="0" />
-  <material name="blue">
-    <color rgba="0 0 0.8 1"/>
-  </material>
-  <material name="white">
-    <color rgba="1 1 1 1"/>
-  </material>
-  <material name="orange">
-    <color rgba="179.0 107.0 0.0 1.0"/>
-  </material>
+  <!-- Import all Gazebo-customisation elements, including Gazebo colours. -->
+  <xacro:include filename="$(find pan_tilt_description)/urdf/pan_tilt.gazebo" />
+  <!-- Import Rviz colours. -->
+  <xacro:include filename="$(find pan_tilt_description)/urdf/materials.xacro" />
   <link name="world"/>
   <!-- Description of base. -->

Commit message: Adding revolute head joint to xacro description.

File: catkin_ws/src/pan_tilt_description/urdf/pan_tilt.urdf.xacro (robot description, xacro)
@@ -151,7 +151,9 @@
   <!-- Roll is around x, yaw is around z, and pitch is around y. -->
   <!-- Connect head with base which allows the head to move in 3D. -->
-  <joint name="head_to_base" type="fixed">
+  <joint name="head_to_base" type="revolute">
     <parent link="base_link" />
     <child link="head_link" />
+    <limit effort="1000.0" lower="-1.571" upper="1.571" velocity="0.5"/>
+	  <axis xyz="0 0 1"/>
     <origin xyz="0 0 0.68" />
   </joint>

Commit message: Adding gazebo-ros-control however a issue #2 is preventing joint control in gazebo through ros.

File: catkin_ws/src/pan_tilt_description/urdf/pan_tilt.urdf.xacro (robot description, xacro)
@@ -1,4 +1,4 @@
 <?xml version="1.0"?>
-<robot xmlns:xacro="http://www.ros.org/wiki/xacro" name="pan_tilt">
+<robot xmlns:xacro="http://www.ros.org/wiki/xacro" name="pan_tilt_bot">
   <!--
   IMPORTANT!
@@ -158,3 +158,15 @@
     <origin xyz="0 0 0.68" />
   </joint>
+  <!-- Use transmission to link motor to head joint. -->
+  <transmission name="transmission1">
+    <!-- Gazebo only supports transmission_interface/SimpleTransmission -->
+    <type>transmission_interface/SimpleTransmission</type>
+    <joint name="head_to_base">
+      <hardwareInterface>EffortJointInterface</hardwareInterface>
+    </joint>
+    <actuator name="actuator1">
+      <hardwareInterface>EffortJointInterface</hardwareInterface>
+      <mechanicalReduction>1</mechanicalReduction>
+    </actuator>
+  </transmission>
 </robot>

Commit message: Changing spawn location of robot in simulation.

File: catkin_ws/src/pan_tilt_description/urdf/pan_tilt.urdf.xacro (robot description, xacro)
@@ -71,5 +71,5 @@
         <box size="${head_link_size_x} ${head_link_size_y} ${head_link_size_z}" />
       </geometry>
-      <origin rpy="0 1.57075 0" xyz="${head_link_origin_x} ${head_link_origin_y} ${head_link_origin_z}"/>
+      <origin rpy="0 0 0" xyz="${head_link_origin_x} ${head_link_origin_y} ${head_link_origin_z}"/>
     </collision>
     <visual>
@@ -77,5 +77,5 @@
         <box size="${head_link_size_x} ${head_link_size_y} ${head_link_size_z}" />
       </geometry>
-      <origin rpy="0 1.57075 0" xyz="${head_link_origin_x} ${head_link_origin_y} ${head_link_origin_z}"/>
+      <origin rpy="0 0 0" xyz="${head_link_origin_x} ${head_link_origin_y} ${head_link_origin_z}"/>
       <material name="orange" />
     </visual>

Commit message: Adding sample Gazebo plugins.

File: catkin_ws/src/pan_tilt_description/urdf/pan_tilt.urdf.xacro (robot description, xacro)
@@ -154,5 +154,5 @@
     <parent link="base_link" />
     <child link="head_link" />
-    <limit effort="1000.0" lower="-1.571" upper="1.571" velocity="0.5"/>
+    <limit effort="1000.0" lower="-1.571" upper="1.571" velocity="5.0"/>
 	  <axis xyz="0 0 1"/>
     <origin xyz="0 0 0.68" />
