Commit message: renamed urdf model files

File: catkin_wsu/src/ur_world_objects/objects/ur5_on_table.urdf.xacro (robot description, xacro)
@@ -4,9 +4,9 @@
   <!-- common stuff -->
   <!--xacro:include filename="$(find ur_description)/urdf/common.gazebo.xacro" /-->
-  <property name="ur_x_offset" value="0.2" />
-  <property name="ur_y_offset" value="-0.2" />
-  <property name="ur_z_offset" value="0.025" />
+  <property name="ur_x_table_offset" value="0.2" />
+  <property name="ur_y_table_offset" value="-0.2" />
+  <property name="ur_z_table_offset" value="0.025" />
   <!-- ur5 -->
-  <xacro:include filename="$(find ur_world_objects)/objects/ur5_robot_on_table.xacro" />
+  <xacro:include filename="$(find ur_world_objects)/objects/ur5_robot.xacro" />
   <!-- Table -->
   <xacro:include filename="$(find ur_world_objects)/objects/table.xacro"/>
@@ -22,5 +22,5 @@
     <parent link="table_top_link" />
     <child link = "base_link" />
-    <origin xyz="${ur_x_offset+table_x-table_width/2} ${ur_y_offset+table_y+table_depth/2} ${ur_z_offset+table_z+table_height}" rpy="0.0 0.0 0.0" />
+    <origin xyz="${ur_x_table_offset+table_x-table_width/2} ${ur_y_table_offset+table_y+table_depth/2} ${ur_z_table_offset+table_z+table_height}" rpy="0.0 0.0 0.0" />
   </joint>
 </robot>
