Commit message: Added gazebo implementation, can now view from camera

File: catkin_ws/src/kinect_description/urdf/kinect.urdf (robot description, URDF)
Before this commit: robot pan_tilt_bot, 5 links, 4 joints
Links:
- removed link base_link
- removed link camera_link_left
- removed link camera_link_right
- removed link head_link
- added link kinect_link, mass 1; collision box size=0.2 0.05 0.05; visual box size=0.2 0.05 0.05
- added link platform_link, mass 1; collision box size=0.4 0.4 0.5; visual box size=0.4 0.4 0.5
- added link sensor, mass 1e-5; collision box size=0.02 0.02 0.02; visual box size=0.02 0.02 0.02
Joints:
- removed joint base_to_world
- removed joint head_to_base
- removed joint left_cam_to_head
- removed joint right_cam_to_head
- added joint kinect_to_platform: type fixed, parent platform_link, child kinect_link
- added joint platform_to_world: type fixed, parent world, child platform_link
- added joint sensor_to_kinect: type fixed, parent kinect_link, child sensor, origin xyz=0.063 -0.035 0.035 rpy=0 0 0, axis 0 1 0

File: catkin_ws/src/kinect_description/urdf/kinect.urdf.xacro (robot description, xacro)
@@ -77,5 +77,5 @@
     </inertial>
   </link>
-  <!-- Description of camera.-->
+  <!-- Description of sensor.-->
   <link name="sensor">
     <collision>

Commit message: Worked on kinect simulation, need to fix depth camera

File: catkin_ws/src/kinect_description/urdf/kinect.urdf (robot description, URDF)
Before this commit: robot kinect_bot, 4 links, 3 joints
Links:
- added link camera, mass 1e-5; collision box size=0.02 0.02 0.02; visual box size=0.02 0.02 0.02
Joints:
- added joint camera_to_kinect: type fixed, parent kinect_link, child camera, origin xyz=-0.063 -0.035 0.035 rpy=0 0 0, axis 0 1 0

File: catkin_ws/src/kinect_description/urdf/kinect.urdf.xacro (robot description, xacro)
@@ -97,4 +97,24 @@
     </inertial>
   </link>
+  <!-- Description of camera.-->
+  <link name="camera">
+    <collision>
+      <geometry>
+        <box size="${camera_link} ${camera_link} ${camera_link}"/>
+      </geometry>
+    </collision>
+    <visual>
+      <geometry>
+         <box size="${camera_link} ${camera_link} ${camera_link}"/>
+      </geometry>
+      <origin rpy="0 0 0" xyz="0 0 0.4875"/>
+       <material name="white" />
+    </visual>
+    <inertial>
+      <mass value="1e-5" />
+      <inertia ixx="1e-6" ixy="0" ixz="0" iyy="1e-6" iyz="0" izz="1e-6" />
+      <origin xyz="0 0 0" rpy="0 0 0" />
+    </inertial>
+  </link>
   <!-- Attach platform to world. -->
   <joint name="platform_to_world" type="fixed">
@@ -115,3 +135,11 @@
     <child link="sensor" />
   </joint>
+  <!-- Attach camera to the kinect. -->
+  <joint name="camera_to_kinect" type="fixed">
+    <axis xyz="0 1 0" />
+    <!-- Determine measurements xyz. -->
+    <origin rpy="0 0 0" xyz="-0.063 -0.035 0.035" />
+    <parent link="kinect_link" />
+    <child link="camera" />
+  </joint>
 </robot>
